File: eagle/afficheur7Segments/interface.sch (EAGLE design)
At the start: 15 parts, among them IC2 MEGA48/88/168-AU, Q1 HC49SM-20-30-50-60-16-ATF

Commit message: I forgot about git syncing :/
Parts:
- removed H1, H2: MOUNT-HOLE2.8, holes:MOUNT-HOLE2.8
- removed Q1: HC49SM-20-30-50-60-16-ATF, crystal:CRYSTALHC49UP
- added C1: 100nF, rcl:C-EUC0805
- added QUARTZ: HC49SM-20, crystal:CRYSTALHC49UP
- added R2, R3, R4, R5, R6: 220, rcl:R-EU_R0805
- ATMEGA328P: value MEGA48/88/168-AU -> ATMEGA328P
- renumbered IC2 to ATMEGA328P, ISP1 to ISP, SV2 to I2C-RXTX
Connections:
- new net N$3: DIS2.CA, R3.1
- new net N$4: DIS3.CA, R4.1
- new net N$5: LED2.C, R5.2
- new net N$6: DIS1.CA, R2.1
- new net N$7: LED1.C, R6.2
- net +5V: now also C1.1, R1.1
- net A: now also ATMEGA328P.PC3(ADC3/PCINT11); no longer ATMEGA328P.PD2(INT0/PCINT18)
- net B: now also ATMEGA328P.PD2(INT0/PCINT18); no longer ATMEGA328P.PD3(INT1/OC2B/PCINT19)
- net C: now also ATMEGA328P.PB1(OC1A/PCINT1); no longer ATMEGA328P.PC0(ADC0/PCINT8)
- net E: now also ATMEGA328P.PC1(ADC1/PCINT9); no longer ATMEGA328P.PC3(ADC3/PCINT11)
- net G: now also ATMEGA328P.PD3(INT1/OC2B/PCINT19); no longer ATMEGA328P.PD5(T1/OC0B/PCINT21)
- net GND: now also C1.2; no longer R1.1
- net L1: now also ATMEGA328P.PC0(ADC0/PCINT8), R2.2; no longer ATMEGA328P.PC1(ADC1/PCINT9), DIS1.CA
- net L2: now also R3.2; no longer DIS2.CA
- net L3: now also R4.2; no longer DIS3.CA
- net LED1: now also ATMEGA328P.PD7(AIN1/PCINT23), R6.1; no longer ATMEGA328P.PB0(ICP1/CLKO/PCINT0), LED1.C
- net LED2: now also ATMEGA328P.PB0(ICP1/CLKO/PCINT0), R5.1; no longer ATMEGA328P.PB1(OC1A/PCINT1), LED2.C
- net N$1: now also ATMEGA328P.PB7(XTAL2/TOSC2/PCINT7), QUARTZ.2; no longer ATMEGA328P.PB6(XTAL1/TOSC1/PCINT6), Q1.2
- net N$2: now also ATMEGA328P.PB6(XTAL1/TOSC1/PCINT6), QUARTZ.1; no longer ATMEGA328P.PB7(XTAL2/TOSC2/PCINT7), Q1.1
Other:
- moved on the sheet: C4, C5
